Commit message: hierarchical registration added

File: assets/ycb_objects/YcbPowerDrill/model.urdf (robot description, URDF)
Before this commit: robot model.urdf, 1 links, 0 joints
Links:
- link baseLink: geometry collision mesh filename=collision_vhacd_1.obj scale=1 1 1; visual mesh filename=textured_simple_reoriented_1.obj scale=1 1 1
